File: Beal-TX/power.kicad_sch (KiCad schematic)
At the start: 28 parts, among them J5 UJ20-C-H-G-MSMT-4B-P16-TR, U150 LM5157-Q1, U2 TPSM863253

Commit message: Beal TX: Address some issues found during prototyping phase
Basically, the prototyping phase has highlighted some issues.
The major one is about the power delivered by an USB-C battery
is not enough to safely driver the valve.
The power after 9V decrease to about 5V, and the 5V from battery
fall to 2.0V.

One way for fixing it is using super capacitor.
This adds an extra cost to the BOM, and, I am not about its
duration regarding the operating conditions.

Because of the cost and the doubt about the longevity,
I would like to evaluate other solutions.
But, we also need to move forward so I made some changes to
power to make it more configurable so we could later try external
battery with a BMS, with different voltage with or without the booster.
By default we will have the super capacitor but we could slit main and
super capacitor board and plug a battery or any power source instead.

A minor change also introduced by this commit is adding testpoints.
Since the hardware an the software is not yet done, testpoints will
be very useful for debugging.

Signed-off-by: Alexandre Bailon <abailon@baylibre.com>
Parts:
- removed C31: 10nF, Capacitor_SMD:C_0402_1005Metric, symbol Device:C
- added J10, J14, J15: Conn_01x03, Connector_PinHeader_2.54mm:PinHeader_1x03_P2.54mm_Vertical, symbol Connector_Generic:Conn_01x03
- added J13: Screw_Terminal_01x03, TerminalBlock_Phoenix:TerminalBlock_Phoenix_MKDS-1,5-3_1x03_P5.00mm_Horizontal, symbol Connector:Screw_Terminal_01x03
- added J2, J8: Conn_01x02, Connector_PinHeader_2.54mm:PinHeader_1x02_P2.54mm_Vertical, symbol Connector_Generic:Conn_01x02
- added R11: 143k, Resistor_SMD:R_0402_1005Metric, symbol Device:R
- added R12: 66.5k, Resistor_SMD:R_0402_1005Metric, symbol Device:R
- added TP1, TP2, TP3, TP4, TP5, TP6, TP7, TP8: TestPoint, TestPoint:TestPoint_Pad_D1.0mm, symbol Connector:TestPoint
- C30: value 10nF -> 4.7uF; MPN GRM155R70J103KA01D -> 4.7uF 16V; Manufacturer_Part_Number GRM155R70J103KA01D -> 4.7uF 16V
- J5: footprint UJ20CHGMSMT4BP16TR -> LIB_UJ20-C-H-G-MSMT-4B-P16-TR/:UJ20CHGMSMT4BP16TR
- U150: footprint Beal:WQFN-16-1EP_3x3mm_P0.5mm_EP1.68x1.68mm_ThermalVias -> Package_DFN_QFN:WQFN-16-1EP_3x3mm_P0.5mm_EP1.68x1.68mm_ThermalVias
Connections:
- net +3.3V: now also TP6.1
- net +9V: now also J10.1 (Pin_1), J15.3 (Pin_3), J2.2 (Pin_2), TP4.1; no longer C2.1, C32.1, C33.1, D6.1 (K), R25.1
- net 9V_EN: now also R11.2, R12.1, TP2.1
- net GND: now also U150.11 (MODE), J13.1 (Pin_1), R12.2, TP7.1, TP8.1
- net VBUS: now also J10.3 (Pin_3), J14.1 (Pin_1), J8.1 (Pin_1); no longer C1.1, C28.2, C6.1, C7.1, L4.1, R3.1, U150.3 (BIAS), U2.1 (VIN)
- net at U150.5 (RT): now also R24.1
- new net: C6.1, C7.1, J10.2 (Pin_2), R3.1, TP5.1, U2.1 (VIN)
- new net: C1.1, C28.2, J15.1 (Pin_1), J8.2 (Pin_2), L4.1, R11.1, TP1.1, U150.3 (BIAS)
- new net: J13.2 (Pin_2), J15.2 (Pin_2)
- new net: J13.3 (Pin_3), J14.2 (Pin_2)
- new net +9V_Boost: C2.1, C32.1, C33.1, D6.1 (K), J14.3 (Pin_3), J2.1 (Pin_1), R25.1, TP3.1
Other:
- note added: "1-2: 3.2V from battery used as input of 9V 2-3: 9V from super capa used to provide 9V"
- note added: "1-2: USB-C used to charge 3.2 battery 2-3: 9V from boost used to charge super capa"
- note added: "1-2: Use 9V as input for 3.3V regulator 2-3: Use VBUS as input for 3.3V regulator"
- note added: "1-2: connect 9V directly to output of buck boost"
- note added: "1-2: connect VBUS directly to input of buck boost"
- note added: "1: GND 2: Ouptut from battery or from super capa 3: Power input, to charge the super capa or the battery"
- note added: "Make sure to stop 9V in case where input voltage drop to much. The motor driver will report an undervoltage error to MCU."
- moved on the sheet: C28, C9, R24

Commit message: Beal-TX: Remove changes previoulsy done regarding done regarding battery tests
I made some measurement on comptitor product and finaly,
the signal to control the valve is not that bad.
I have decided to just add a capacitor and to remove all the
tests features added by previous commit.

This also tries to address some potential issues and does some
improvements such as increasing traces for VBUS and +9V.

Signed-off-by: Alexandre Bailon <abailon@baylibre.com>
Parts:
- removed J10, J14, J15: Conn_01x03, Connector_PinHeader_2.54mm:PinHeader_1x03_P2.54mm_Vertical, symbol Connector_Generic:Conn_01x03
- removed J13: Screw_Terminal_01x03, TerminalBlock_Phoenix:TerminalBlock_Phoenix_MKDS-1,5-3_1x03_P5.00mm_Horizontal, symbol Connector:Screw_Terminal_01x03
- removed J2, J8: Conn_01x02, Connector_PinHeader_2.54mm:PinHeader_1x02_P2.54mm_Vertical, symbol Connector_Generic:Conn_01x02
- removed TP4, TP5: TestPoint, TestPoint:TestPoint_Pad_D1.0mm, symbol Connector:TestPoint
- C27: value 23uF -> 22uF
Connections:
- net +9V_Boost is gone; now on net +9V: C2.1, C32.1, C33.1, D6.1 (K), R25.1, TP3.1
- net GND: now also J5.MH1 (MH_1), J5.MH2 (MH_2), J5.MH3 (MH_3), J5.MH4 (MH_4)
- net VBUS: now also C1.1, C28.2, C6.1, C7.1, L4.1, R11.1, R3.1, TP1.1, U150.3 (BIAS), U2.1 (VIN)
- no-connect marks 12 -> 8
Other:
- note removed: "1-2: 3.2V from battery used as input of 9V 2-3: 9V from super capa used to provide 9V"
- note removed: "1-2: USB-C used to charge 3.2 battery 2-3: 9V from boost used to charge super capa"
- note removed: "1-2: Use 9V as input for 3.3V regulator 2-3: Use VBUS as input for 3.3V regulator"
- note removed: "1-2: connect 9V directly to output of buck boost"
- note removed: "1-2: connect VBUS directly to input of buck boost"
- note removed: "1: GND 2: Ouptut from battery or from super capa 3: Power input, to charge the super capa or the battery"
- note removed: "Make sure to stop 9V in case where input voltage drop to much. The motor driver will report an undervoltage error to MCU."
