File: Beal-TX/radio_mcu.kicad_sch (KiCad schematic)
At the start: 23 parts, among them J1 CONMHF1-SMD-T, J3 Conn_02x04_Odd_Even, J4 Conn_02x04_Odd_Even, J7 TC2050, SW2 SW_Push, U5 LoRa-E5

Commit message: Beal TX: Address some issues found during prototyping phase
Basically, the prototyping phase has highlighted some issues.
The major one is about the power delivered by an USB-C battery
is not enough to safely driver the valve.
The power after 9V decrease to about 5V, and the 5V from battery
fall to 2.0V.

One way for fixing it is using super capacitor.
This adds an extra cost to the BOM, and, I am not about its
duration regarding the operating conditions.

Because of the cost and the doubt about the longevity,
I would like to evaluate other solutions.
But, we also need to move forward so I made some changes to
power to make it more configurable so we could later try external
battery with a BMS, with different voltage with or without the booster.
By default we will have the super capacitor but we could slit main and
super capacitor board and plug a battery or any power source instead.

A minor change also introduced by this commit is adding testpoints.
Since the hardware an the software is not yet done, testpoints will
be very useful for debugging.

Signed-off-by: Alexandre Bailon <abailon@baylibre.com>
Parts:
- added TP10, TP11, TP12, TP21, TP22, TP9: TestPoint, TestPoint:TestPoint_Pad_D1.0mm, symbol Connector:TestPoint
- J1: footprint CONMHF1SMDT -> CONMHF1-SMD-T:CONMHF1SMDT
Connections:
- net E5_RX: now also TP22.1
- net E5_TX: now also TP21.1
- net I2C_INT0: now also TP11.1
- net I2C_INT1: now also TP12.1
- net SCL: now also TP10.1
- net SDA: now also TP9.1

Commit message: Beal-TX: Remove changes previoulsy done regarding done regarding battery tests
I made some measurement on comptitor product and finaly,
the signal to control the valve is not that bad.
I have decided to just add a capacitor and to remove all the
tests features added by previous commit.

This also tries to address some potential issues and does some
improvements such as increasing traces for VBUS and +9V.

Signed-off-by: Alexandre Bailon <abailon@baylibre.com>
Parts:
- added R17, R28: 0, Resistor_SMD:R_0402_1005Metric, symbol Device:R
- C5: MPN 10uF 16V 0805 -> 0.1uF 16V 0805
- L2: MPN RC0603FR-100RL -> 0201WMF0000TEE
Connections:
- net +3.3V: now also R23.1; no longer C25.1
- net E5_RX: now also R17.2; no longer J7.8
- net E5_TX: now also R28.2; no longer J7.9
- net GND: now also C25.2; no longer R23.2
- net MCU_FAULT_N: now also U5.13 (PC0); no longer U5.28 (PB0)
- net WIO_RESET: now also C25.1, R23.2; no longer C25.2, R23.1
- net at J7.7: now also R28.1
- new net: J7.8, R17.1
Other:
- moved on the sheet: TP21, TP22
